File: PCB/KiCAD/PhobGCC_2_0_2_round.kicad_pcb (KiCad board)
At the start: 2 copper layers, 125.5 x 90.3 mm, 108 parts, among them J1 Conn_01x06_Female, J11 Conn_01x02, J14 Conn_01x06, J15 Conn_01x06, J2 Conn_01x02, J3 Conn_01x02, J4 Conn_01x01, J5 Rumble, J6 Conn_01x06, J8 USB_B_Micro, Q1 Q_NMOS_GSD, Q2 Q_PMOS_GDS, Q3 Q_NMOS_GSD, SW1 A, SW10 Dup, SW11 Dright, SW12 Ddown, SW2 B, SW3 X, SW4 Y, SW5 Start, SW6 L, SW7 R, SW8 Z, SW9 Dleft, U1 MCP3002, U10 DRV5055A2xDBZxQ1, U11 DRV5055A2xDBZxQ1, U2 Stickbox_Assembly_Main, U3 MCP3002, U4 DRV5055A2xDBZxQ1, U5 Stickbox_Assembly_CStick, U6 AMS1117-3.3, U7 W25Q128JVS, U8 RP2040, U9 DRV5055A2xDBZxQ1, Y1 Crystal_GND24

Commit message: added version with no round
Parts:
- removed the G*** at (111.9, 91.1)
- removed the G*** at (54.7, 46.3)
- removed the G*** at (150.1, 37.7)
- added G***: LOGO, CrossBlack:10 Circle, F.Cu at (54.3, 46.0)
- added G***: LOGO, CrossBlack:6 Circle, F.Cu at (111.8, 91.4)
- added G***: LOGO, CrossBlack:29,5 Circle, B.Cu at (88.9, 80.8)
- added G***: LOGO, CrossBlack:10 Circle, B.Cu at (149.9, 37.0)
- moved J5 2.15 mm to (88.3, 69.1)
Routing:
- net +5V: track 152.8 -> 155.0 mm
- net Net-(D2-Pad2): track 88.9 -> 91.0 mm
